File: ESPBoatSchematic/ESPBoatSchematic.kicad_sch (KiCad schematic)
At the start: 1 part, among them U1 ESP32-DEVKITC-32D

Commit message: First commit. We'll see if this works
Parts:
- added Adafruit-MPU6050: ~, symbol New_Library:Adafruit-MPU6050.SM
- added J1: XT60-M, XT60-M:AMASS_XT60-M, symbol XT60-M:XT60-M
- added U3: GT-U7, GT-U7_GPS-Module:GT-U7_SMT, symbol GT-U7_GPS-Module:GT-U7_GPS_Module
Connections:
- net XBee_RX: now reaches U1.J2-10 (IO26)
- net GND: now reaches U1.J2-14 (GND1)
- net GND: now also Adafruit-MPU6050. (VIN), U3.2 (GND)
- net +5V: now reaches U1.J2-19 (EXT_5V)
- net +5V: now also Adafruit-MPU6050. (VIN), U3.1 (VCC)
- net XBee_TX: now reaches U1.J2-9 (IO25)
- net at U1.J3-11 (IO17): now also U3.3 (RXD)
- net at U1.J3-12 (IO16): now also U3.4 (TXD)
- net I2C_SCL: now reaches U1.J3-3 (IO22)
- net I2C_SDA: now reaches U1.J3-6 (IO21)
- net Tail_PWM: now reaches U1.J3-8 (IO19)
- net Sail_PWM: now reaches U1.J3-9 (IO18)
Other:
- note added: "I2C Bus"
- note added: "Outputs"
- note added: "Power Module"
- note added: "To make things compact, let's try making our own DC-DC buck converter"
- moved on the sheet: U1

Commit message: Update schematic
Parts:
- added Adafruit-LIS3MDL: ~, symbol New_Library:TAF-Adafruit-LIS3MDL
- added J2: 2140940040, CONN4_214094-0040_MOL, symbol 2024-11-02_12-47-29:2140940040
- added J3, J4, J5: 2140940030, CONN_214094-0030_MOL, symbol 2024-11-02_12-53-35:2140940030
Connections:
- net +5V: now also Adafruit-LIS3MDL. (Vin), J2.1, J3.2, J4.2, J5.2
- net GND: now also Adafruit-LIS3MDL. (Vin), J2.4, J3.1, J4.1, J5.1
- net I2C_SCL: now also Adafruit-MPU6050. (VIN), Adafruit-LIS3MDL. (Vin), J2.3
- net I2C_SDA: now also Adafruit-MPU6050. (VIN), Adafruit-LIS3MDL. (Vin), J2.2
- net Sail_PWM: now also J4.3
- net Tail_PWM: now also J3.3
- net Water_Sense: now reaches U1.J2-3 (SENSOR_VP)
- net Water_Sense: now also J5.3
- no-connect marks 0 -> 34
Other:
- note added: "Board integrated Xbee breakout so we don't need to keep buying them."
- note added: "Sail Servo Out"
- note added: "Tail Servo Out"
- note added: "Water Sense Out"
- note added: "Windvane Out"
- note added: "Xbee Module"
